File: Electrical/Transistor/eCAD/Eboard.sch (EAGLE design)
At the start: 22 parts

Commit message: added gnd pin to encoders
Connections:
- removed net N$3: STEER_ENC.4
- net GND: now also STEER_ENC.4
Changed lines of the file:
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@@
 <part name="SUPPLY6" library="SparkFun-Aesthetics" deviceset="5V" device=""/>
 <part name="SERVO_MTR" library="SparkFun-Connectors" library_urn="urn:adsk.eagle:library:513" deviceset="CONN_02" device="" package3d_urn="urn:adsk.eagle:package:38039/1"/>
+<part name="GND12" library="SparkFun-PowerSymbols" library_urn="urn:adsk.eagle:library:530" deviceset="GND" device=""/>
 </parts>
 <sheets>
@@
 <instance part="SUPPLY6" gate="G$1" x="213.36" y="86.36"/>
 <instance part="SERVO_MTR" gate="G$1" x="182.88" y="76.2" rot="R180"/>
+<instance part="GND12" gate="1" x="205.74" y="63.5"/>
 </instances>
 <busses>
@@
 <wire x1="200.66" y1="119.38" x2="200.66" y2="116.84" width="0.1524" layer="91"/>
 </segment>
+<segment>
+<pinref part="STEER_ENC" gate="A" pin="4"/>
+<wire x1="200.66" y1="73.66" x2="205.74" y2="73.66" width="0.1524" layer="91"/>
+<wire x1="205.74" y1="73.66" x2="205.74" y2="66.04" width="0.1524" layer="91"/>
+<pinref part="GND12" gate="1" pin="GND"/>
+</segment>
 </net>
 <net name="12V" class="0">
@@
 </segment>
 </net>
-<net name="N$3" class="0">
-<segment>
-<pinref part="STEER_ENC" gate="A" pin="4"/>
-<wire x1="195.58" y1="73.66" x2="200.66" y2="73.66" width="0.1524" layer="91"/>
-</segment>
-</net>
